Commit message: added fire wtih temp and heat cam but fire heat signature doesnt work yet

File: simulations/41068_ignition_bringup/urdf_drone/parrot.gazebo.xacro (robot description, xacro)
@@ -165,3 +165,30 @@
     </sensor>
   </gazebo>
+  <!-- IR Thermal Camera -->
+  <gazebo reference="ir_camera_link">
+    <sensor name="ir_camera" type="thermal_camera">
+      <camera>
+        <horizontal_fov>1.047</horizontal_fov>
+        <image>
+          <width>1080</width>
+          <height>720</height>
+          <format>L8</format>  <!-- 8-bit grayscale for thermal -->
+        </image>
+        <clip>
+          <near>0.1</near>
+          <far>50.0</far>
+        </clip>
+      </camera>
+      <thermal_camera>
+        <temperature_range>
+          <min>250.0</min>  <!-- -23°C -->
+          <max>700.0</max>  <!-- 427°C -->
+        </temperature_range>
+      </thermal_camera>
+      <always_on>1</always_on>
+      <update_rate>15</update_rate>
+      <topic>model/drone/ir_camera</topic>
+      <gz_frame_id>ir_camera_link</gz_frame_id>
+    </sensor>
+  </gazebo>
 </robot>

File: simulations/41068_ignition_bringup/urdf_drone/parrot.urdf.xacro (robot description, xacro)
@@ -124,3 +124,27 @@
   </joint>
   <link name="camera_depth_optical_frame"/>
+  <!-- IR Camera Link -->
+<link name="ir_camera_link">
+  <visual>
+    <geometry>
+      <box size="0.05 0.05 0.03"/>
+    </geometry>
+    <material name="black"/>
+  </visual>
+  <collision>
+    <geometry>
+      <box size="0.05 0.05 0.03"/>
+    </geometry>
+  </collision>
+  <inertial>
+    <mass value="0.1"/>
+    <inertia ixx="0.001" ixy="0" ixz="0" iyy="0.001" iyz="0" izz="0.001"/>
+  </inertial>
+</link>
+<!-- Joint to attach camera to bottom of drone -->
+<joint name="ir_camera_joint" type="fixed">
+  <parent link="base_link"/>
+  <child link="ir_camera_link"/>
+  <origin xyz="0 0 -0.1" rpy="0 ${pi/2} 0"/>  <!-- Pointing downward -->
+</joint>
 </robot>

Commit message: changed world to spawn fire infront + rviz setup

File: simulations/41068_ignition_bringup/urdf_drone/parrot.gazebo.xacro (robot description, xacro)
@@ -171,7 +171,7 @@
         <horizontal_fov>1.047</horizontal_fov>
         <image>
-          <width>1080</width>
-          <height>720</height>
-          <format>L16</format>  <!-- 8-bit grayscale for thermal -->
+          <width>320</width>
+          <height>240</height>
+          <format>R8G8B8</format>  <!-- RGB format for thermal visualization -->
         </image>
         <clip>
@@ -182,7 +182,8 @@
       <thermal_camera>
         <temperature_range>
-          <min>250.0</min>  <!-- -23°C -->
-          <max>700.0</max>  <!-- 427°C -->
+          <min>253.15</min>  <!-- -20°C in Kelvin -->
+          <max>773.15</max>  <!-- 500°C in Kelvin -->
         </temperature_range>
+        <temperature_linear_resolution>0.01</temperature_linear_resolution>
       </thermal_camera>
       <always_on>1</always_on>

File: simulations/41068_ignition_bringup/urdf_drone/parrot.urdf.xacro (robot description, xacro)
@@ -146,5 +146,5 @@
   <parent link="base_link"/>
   <child link="ir_camera_link"/>
-  <origin xyz="0 0 -0.1" rpy="0 ${pi/2} 0"/>  <!-- Pointing downward -->
+  <origin xyz="0 0 -0.1" rpy="0 0 0"/>  <!-- SDF camera looks along -Z; this points down -->
 </joint>
 </robot>

Commit message: Fixed lots of stuff

File: simulations/41068_ignition_bringup/urdf_drone/parrot.gazebo.xacro (robot description, xacro)
@@ -5,4 +5,11 @@
   <xacro:arg name="imu_visual"    default="false"/>
   <!-- <xacro:include filename="$(find 41068_ignition_bringup)/urdf/wheel.urdf.xacro"/> -->
+  <!-- Physics properties for base_link to ensure proper motion -->
+  <gazebo reference="base_link">
+    <gravity>1</gravity>
+    <mu1>0.1</mu1>
+    <mu2>0.1</mu2>
+    <material>Gazebo/DarkGrey</material>
+  </gazebo>
   <gazebo reference="imu_link">
     <sensor type="imu" name="imu">
@@ -79,15 +86,26 @@
       name="ignition::gazebo::systems::VelocityControl">
       <topic>model/drone/cmd_vel</topic>
+      <enable_3d>true</enable_3d>
+      <linear_velocity>
+        <x>1</x>
+        <y>1</y>
+        <z>1</z>
+      </linear_velocity>
+      <angular_velocity>
+        <x>1</x>
+        <y>1</y>
+        <z>1</z>
+      </angular_velocity>
     </plugin>
   </gazebo>
-  <!-- Publish odometry separately -->
+  <!-- Publish odometry using model plugin approach -->
   <gazebo>
     <plugin
       filename="ignition-gazebo-odometry-publisher-system"
       name="ignition::gazebo::systems::OdometryPublisher">
-      <topic>model/drone/odometry</topic>
-      <odom_publish_frequency>20</odom_publish_frequency>
       <odom_frame>odom</odom_frame>
       <robot_base_frame>base_link</robot_base_frame>
+      <odom_topic>model/drone/odometry</odom_topic>
+      <odom_publish_frequency>20</odom_publish_frequency>
     </plugin>
   </gazebo>
@@ -96,5 +114,5 @@
       filename="ignition-gazebo-joint-state-publisher-system"
       name="ignition::gazebo::systems::JointStatePublisher">
-      <topic>model/husky/joint_states</topic>
+      <topic>model/drone/joint_states</topic>
     </plugin>
   </gazebo>
@@ -137,6 +155,6 @@
         <horizontal_fov>2.0944</horizontal_fov>
         <image>
-          <width>720</width>
-          <height>480</height>
+          <width>1280</width>
+          <height>720</height>
         </image>
         <clip>
@@ -188,5 +206,5 @@
       </thermal_camera>
       <always_on>1</always_on>
-      <update_rate>15</update_rate>
+      <update_rate>2</update_rate>  <!-- Reduced from 15 to 2 Hz to prevent lag -->
       <visualize>true</visualize>
       <topic>/model/drone/ir_camera</topic>

File: simulations/41068_ignition_bringup/urdf_drone/parrot.urdf.xacro (robot description, xacro)
@@ -16,10 +16,10 @@
                izz="3.328e-3" />
     </inertial>
-<!--     <collision name="collision">
-      <origin xyz="-0.00424 0.00014 -0.00595" rpy="0 0 0"/>
-      <geometry>
-        <box size="0.5 0.5 0.2"/>
-      </geometry>
-    </collision> -->
+    <collision name="collision">
+      <origin xyz="0 0 0" rpy="0 0 0"/>
+      <geometry>
+        <box size="0.3 0.3 0.1"/>
+      </geometry>
+    </collision>
     <visual name="hull">
       <geometry>
@@ -80,5 +80,5 @@
   </link>
   <joint name="camera_joint" type="fixed">
-    <origin xyz="0.25 0.0 0.25" rpy="0 0.785398 0"/> <!-- 0.5 0.0 0.9 -->
+    <origin xyz="0.15 0.0 0.1" rpy="0 0 0"/> <!-- Moved closer and higher up on drone -->
     <parent link="base_link"/>
     <child link="camera_link"/>
@@ -142,9 +142,62 @@
   </inertial>
 </link>
-<!-- Joint to attach camera to bottom of drone -->
+<!-- Joint to attach camera to front of drone -->
 <joint name="ir_camera_joint" type="fixed">
   <parent link="base_link"/>
   <child link="ir_camera_link"/>
-  <origin xyz="0 0 -0.1" rpy="0 1.57 0"/>
+  <origin xyz="0.1 0 0.05" rpy="0 0 0"/> <!-- Moved to front and slightly up -->
 </joint>
+  <!-- Propeller Links and Joints for MulticopterVelocityControl -->
+  <!-- Front Left Propeller -->
+  <link name="propeller_fl_link">
+    <inertial>
+      <mass value="0.005"/>
+      <inertia ixx="0.000001" ixy="0" ixz="0" iyy="0.000001" iyz="0" izz="0.000001"/>
+    </inertial>
+  </link>
+  <joint name="propeller_fl_joint" type="continuous">
+    <parent link="base_link"/>
+    <child link="propeller_fl_link"/>
+    <origin xyz="0.08456 0.11463 -0.00501" rpy="0 0 0"/>
+    <axis xyz="0 0 1"/>
+  </joint>
+  <!-- Front Right Propeller -->
+  <link name="propeller_fr_link">
+    <inertial>
+      <mass value="0.005"/>
+      <inertia ixx="0.000001" ixy="0" ixz="0" iyy="0.000001" iyz="0" izz="0.000001"/>
+    </inertial>
+  </link>
+  <joint name="propeller_fr_joint" type="continuous">
+    <parent link="base_link"/>
+    <child link="propeller_fr_link"/>
+    <origin xyz="0.08456 -0.11435 -0.00501" rpy="0 0 0"/>
+    <axis xyz="0 0 1"/>
+  </joint>
+  <!-- Rear Left Propeller -->
+  <link name="propeller_rl_link">
+    <inertial>
+      <mass value="0.005"/>
+      <inertia ixx="0.000001" ixy="0" ixz="0" iyy="0.000001" iyz="0" izz="0.000001"/>
+    </inertial>
+  </link>
+  <joint name="propeller_rl_joint" type="continuous">
+    <parent link="base_link"/>
+    <child link="propeller_rl_link"/>
+    <origin xyz="0.09035 0.11452 -0.00501" rpy="0 0 0"/>
+    <axis xyz="0 0 1"/>
+  </joint>
+  <!-- Rear Right Propeller -->
+  <link name="propeller_rr_link">
+    <inertial>
+      <mass value="0.005"/>
+      <inertia ixx="0.000001" ixy="0" ixz="0" iyy="0.000001" iyz="0" izz="0.000001"/>
+    </inertial>
+  </link>
+  <joint name="propeller_rr_joint" type="continuous">
+    <parent link="base_link"/>
+    <child link="propeller_rr_link"/>
+    <origin xyz="-0.09035 -0.11423 -0.00501" rpy="0 0 0"/>
+    <axis xyz="0 0 1"/>
+  </joint>
 </robot>
