Commit message: fixed drone position

File: simulations/41068_ignition_bringup/urdf_drone/parrot.urdf.xacro (robot description, xacro)
@@ -146,5 +146,5 @@
   <parent link="base_link"/>
   <child link="ir_camera_link"/>
-  <origin xyz="0 0 -0.1" rpy="0 0 0"/>  <!-- SDF camera looks along -Z; this points down -->
+  <origin xyz="0 0 -0.1" rpy="0 1.57 0"/>
 </joint>
 </robot>

Commit message: Fire detection working great

File: simulations/41068_ignition_bringup/urdf_drone/parrot.urdf.xacro (robot description, xacro)
@@ -142,9 +142,9 @@
   </inertial>
 </link>
-<!-- Joint to attach camera to front of drone -->
+<!-- Joint to attach camera underneath drone facing down -->
 <joint name="ir_camera_joint" type="fixed">
   <parent link="base_link"/>
   <child link="ir_camera_link"/>
-  <origin xyz="0.1 0 0.05" rpy="0 0 0"/> <!-- Moved to front and slightly up -->
+  <origin xyz="0 0 -0.05" rpy="0 1.57 0"/> <!-- Moved underneath and rotated to face down -->
 </joint>
   <!-- Propeller Links and Joints for MulticopterVelocityControl -->
