Commit message: Increased slam resolution, reduced husky lidar height

File: simulations/41068_ignition_bringup/urdf/husky.gazebo.xacro (robot description, xacro)
@@ -106,10 +106,10 @@
       <visualize>$(arg laser_visual)</visualize>
       <topic>model/husky/scan</topic>
-      <update_rate>3</update_rate>
+      <update_rate>10</update_rate>
       <gz_frame_id>base_scan</gz_frame_id>
       <ray>
         <scan>
           <horizontal>
-            <samples>360</samples>
+            <samples>720</samples>
             <resolution>1</resolution>
             <min_angle>0.0</min_angle>
@@ -120,5 +120,5 @@
           <min>0.2</min>
           <max>40</max>
-          <resolution>0.015</resolution>
+          <resolution>0.005</resolution>
         </range>
         <noise>

File: simulations/41068_ignition_bringup/urdf/husky.urdf.xacro (robot description, xacro)
@@ -102,5 +102,5 @@
     <parent link="base_link"/>
     <child link="base_scan"/>
-    <origin xyz="0 0 0.68" rpy="0 0 0"/>
+    <origin xyz="0 0 0.4" rpy="0 0 0"/>
   </joint>
   <link name="base_scan">
