Commit message: husky firefihter added, its scuffed, also changes to nav2 settings for husky like its bounding box (read collision fix summary)

File: simulations/41068_ignition_bringup/urdf/husky.urdf.xacro (robot description, xacro)
@@ -102,5 +102,5 @@
     <parent link="base_link"/>
     <child link="base_scan"/>
-    <origin xyz="0 0 0.4" rpy="0 0 0"/>
+    <origin xyz="0 0 0.35" rpy="0 0 0"/>
   </joint>
   <link name="base_scan">

Commit message: Oincreased map res

File: simulations/41068_ignition_bringup/urdf/husky.urdf.xacro (robot description, xacro)
@@ -102,5 +102,5 @@
     <parent link="base_link"/>
     <child link="base_scan"/>
-    <origin xyz="0 0 0.35" rpy="0 0 0"/>
+    <origin xyz="0 0 0.05" rpy="0 0 0"/>
   </joint>
   <link name="base_scan">
